Commit message: fix(robots/panda.urdf): add dummy table for testing of static mesh loading

File: robots/panda.urdf (robot description, URDF)
Before this commit: robot panda, 9 links, 8 joints
Links:
- added link scene_table_link; collision box size=1 1 1; visual box size=1 1 1
- added link scene_world
Joints:
- added joint table_joint: type fixed, parent scene_world, child scene_table_link, origin xyz=1 0 0 rpy=0 0 0
- added joint world_to_robot: type fixed, parent scene_world, child panda_link0, origin xyz=0 0 0 rpy=0 0 0
